File: LE75LRE/LE75LRE.kicad_sch (KiCad schematic)
At the start: 174 parts, among them P1 USB_C_Plug_USB2.0, SW1 SW_Push, U1 ATmega32U4-A, Y1 YSX321SL

Commit message: Low profile variant
Small fixes, added LP variant
Parts:
- S1, S10, S11, S12, S13, S14, S15, S16, S17, S18, S19, S2, S20, S21, S22, S23, S24, S25, S26, S27, S28, S29, S3, S30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: footprint PCM_Switch_Keyboard_Hotswap_Kailh:SW_Hotswap_Kailh_MX_Plated -> Gateron_KS33_Hotswap:Gateron-KS33-Hotswap-1U
