File: LE75RE/LE75RE.kicad_pcb (KiCad board)
At the start: 2 copper layers, 285 x 94.6 mm, 173 parts, among them P1 USB_C_Plug_USB2.0, SW1 SW_Push, U1 ATmega32U4-A, Y1 YSX321SL

Commit message: Low profile variant
Small fixes, added LP variant
Parts:
- added G***: LOGO, LOGO, B.Cu at (212.6, 88.1)
Other:
- board text added: "leenknegt.eu le75re"

Commit message: Many changes
Parts:
- removed R4: 10k, Resistor_SMD:R_0603_1608Metric
- removed Y1: YSX321SL, Crystal:Crystal_SMD_3225-4Pin_3.2x2.5mm
- added C1: 1u, Capacitor_SMD:C_0603_1608Metric, B.Cu at (19.0, 71.2)
- added C10: 4.7u, Capacitor_SMD:C_0603_1608Metric, B.Cu at (30.4, 86.5)
- added C8: 100n, Capacitor_SMD:C_0603_1608Metric, B.Cu at (31.8, 92.4)
- added C9: 100n, Capacitor_SMD:C_0603_1608Metric, B.Cu at (48.2, 92.2)
- added R5: 22, Resistor_SMD:R_0603_1608Metric, B.Cu at (21.8, 57.5)
- added R6: 5.1k, Resistor_SMD:R_0603_1608Metric, B.Cu at (20.1, 58.3)
- added U2: STM32F072CBTx, Package_QFP:LQFP-48_7x7mm_P0.5mm, B.Cu at (37.5, 88.5)
- C2: value .1uF -> 1u
- C3: value 20pF -> 10n
- C4: value 20pF -> 1u
- C5: value 1uF -> 100n
- C6: value .1uF -> 4.7u
- C7: value .1uF -> 100n
- U1: value ATmega32U4-A -> MCP1703Ax-330xxDB; footprint Package_DFN_QFN:QFN-44-1EP_7x7mm_P0.5mm_EP5.2x5.2mm -> Package_TO_SOT_SMD:SOT-223-3_TabPin2
- moved U1 107.0 mm to (13.7, 69.4), turned to 180 degrees
- moved C2 99.5 mm to (16.9, 63.8), turned to 90 degrees
- moved C4 85.6 mm to (40.7, 95.8), turned to 90 degrees
- moved C6 84.6 mm to (38.3, 81.8), turned to -135 degrees
- moved C3 84.1 mm to (42.2, 93.5)
- moved C5 80.3 mm to (36.9, 81.1)
- moved C7 71.4 mm to (44.0, 88.6), turned to 135 degrees
- moved R3 11.4 mm to (30.4, 90.3), turned to -90 degrees
- moved R2 10.0 mm to (26.8, 67.7), turned to 180 degrees
- moved FL1 8.92 mm to (22.9, 66.7), turned to 0 degrees
- moved R1 7.60 mm to (26.8, 65.9), turned to 180 degrees
- moved D33 6.88 mm to (51.3, 92.0)
- renumbered H4 to H7
Connections:
- net Net-(FL1-I/O1-Pad1) renamed usb+
- net Net-(FL1-I/O2-Pad3) renamed usb-
- C2 pad 1: GND -> VBUS
- C2 pad 2: VCC -> GND
- C3 pad 2: /XTAL_N -> VCC
- C4 pad 2: /XTAL_P -> VCC
- C5 pad 2: Net-(U1-UCAP) -> VCC
- F1 pad 1: VCC -> VBUS
- FL1 pad 5: VCC -> VBUS
- P1 pad A5: unconnected-(P1-CC1-PadA5) -> Net-(P1-CC1)
- P1 pad B5: unconnected-(P1-CC2-PadB5) -> Net-(P1-CC2)
- R3 pad 1: Net-(U1-~{RESET}) -> Net-(U2-BOOT0)
- SW1 pad 2: Net-(U1-~{RESET}) -> Net-(U2-BOOT0)
- U1 pad 1: Col 2 -> VBUS
- U1 pad 2: VCC -> GND
- U1 pad 3: /U1_D- -> VCC
Routing:
- net VCC: track 217.1 -> 75.7 mm, vias 8 -> 3
- net Net-(U1-~{RESET}): track 118.6 -> 0.00 mm, vias 2 -> 0
- net /U1_D+: track 131.2 -> 28.8 mm
- net /U1_D-: track 128.6 -> 29.4 mm
- net Col 13: track 220.5 -> 302.2 mm
- net Col 14: track 243.6 -> 321.7 mm
- net Col 0: track 174.0 -> 100.0 mm, vias 1 -> 0
- net Col 12: track 214.6 -> 282.9 mm
- net Col 1: track 154.7 -> 86.5 mm, vias 1 -> 0
- net Col 9: track 159.7 -> 227.2 mm, vias 1 -> 3
- net Col 11: track 196.4 -> 263.5 mm
- net Col 10: track 178.1 -> 244.0 mm
- net Col 6: track 99.2 -> 163.2 mm
- net Col 5: track 82.3 -> 144.6 mm
- net Col 7: track 120.9 -> 183.2 mm, vias 3 -> 1
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