File: Legacy/LE75LRE_Legacy/LE75LRE_Legacy.kicad_pcb (KiCad board)
At the start: 2 copper layers, 285 x 94.6 mm, 179 parts, among them P1 USB_C_Plug_USB2.0, SW1 SW_Push, U1 MCP1703Ax-330xxDB, U2 STM32F072CBTx

Commit message: Many changes
Parts:
- removed C1: 1u, Capacitor_SMD:C_0603_1608Metric
- removed C10: 4.7u, Capacitor_SMD:C_0603_1608Metric
- removed C8, C9: 100n, Capacitor_SMD:C_0603_1608Metric
- removed R5, R6: 5.1k, Resistor_SMD:R_0603_1608Metric
- removed U2: STM32F072CBTx, Package_QFP:LQFP-48_7x7mm_P0.5mm
- added H7: MountingHole, Keebio-Parts:MountingSlot_2.7mm_M2.5_ISO7380, F.Cu at (76.2, 85.7)
- added R4: 10k, Resistor_SMD:R_0603_1608Metric, B.Cu at (108.6, 109.9)
- added Y1: YSX321SL, Crystal:Crystal_SMD_3225-4Pin_3.2x2.5mm, B.Cu at (121.9, 108.0)
- C2: value 1u -> .1uF
- C3: value 10n -> 20pF
- C4: value 1u -> 20pF
- C5: value 100n -> 1uF
- C6: value 4.7u -> .1uF
- C7: value 100n -> .1uF
- U1: value MCP1703Ax-330xxDB -> ATmega32U4-A; footprint Package_TO_SOT_SMD:SOT-223-3_TabPin2 -> Package_DFN_QFN:QFN-44-1EP_7x7mm_P0.5mm_EP5.2x5.2mm
- moved U1 113.0 mm to (114.2, 108.4), turned to -90 degrees
- moved C2 102.4 mm to (108.4, 106.1), turned to 0 degrees
- moved C6 87.0 mm to (117.5, 114.0), turned to 180 degrees
- moved C3 84.6 mm to (125.6, 106.8), turned to 180 degrees
- moved C4 82.7 mm to (125.6, 109.3), turned to 180 degrees
- moved C5 80.1 mm to (115.6, 102.2), turned to 180 degrees
- moved C7 64.2 mm to (111.1, 98.0), turned to -90 degrees
- moved R2 10.8 mm to (17.3, 62.4), turned to 90 degrees
- moved FL1 10.4 mm to (18.1, 58.3), turned to -90 degrees
- moved R1 8.42 mm to (19.1, 62.4), turned to 90 degrees
- moved D51 5.24 mm to (111.1, 116.8)
- moved D32 4.67 mm to (33.3, 92.9), turned to -90 degrees
- moved D33 3.02 mm to (52.4, 92.9)
- moved F1 1.08 mm to (10.8, 53.5)
- renumbered H7 to H4
Connections:
- net usb+ renamed Net-(FL1-I/O1-Pad1)
- net usb- renamed Net-(FL1-I/O2-Pad3)
- C2 pad 1: VBUS -> GND
- C2 pad 2: GND -> VCC
- C3 pad 2: VCC -> /XTAL_N
- C4 pad 2: VCC -> /XTAL_P
- C5 pad 2: VCC -> Net-(U1-UCAP)
- F1 pad 1: VBUS -> VCC
- FL1 pad 5: VBUS -> VCC
- P1 pad A5: Net-(P1-CC1) -> unconnected-(P1-CC1-PadA5)
- P1 pad B5: Net-(P1-CC2) -> unconnected-(P1-CC2-PadB5)
- R3 pad 1: Net-(U2-BOOT0) -> Net-(U1-~{RESET})
- SW1 pad 2: Net-(U2-BOOT0) -> Net-(U1-~{RESET})
- U1 pad 1: VBUS -> Col 2
- U1 pad 2: GND -> VCC
- U1 pad 3: VCC -> /U1_D-
Routing:
- net Net-(U1-~{RESET}): track 0.00 -> 127.0 mm, vias 0 -> 4
- net VCC: track 78.7 -> 205.0 mm, vias 0 -> 8
- net /U1_D+: track 28.6 -> 133.3 mm
- net /U1_D-: track 30.6 -> 130.6 mm
- net Col 13: track 290.5 -> 213.2 mm
- net Col 8: track 192.9 -> 117.1 mm
- net Col 7: track 170.5 -> 98.8 mm, vias 1 -> 0
- net Col 2: track 77.5 -> 145.5 mm
- net Col 0: track 116.8 -> 184.6 mm
- net Col 14: track 309.8 -> 242.4 mm
- net Col 1: track 99.7 -> 164.3 mm
- net Col 12: track 271.0 -> 211.7 mm, vias 1 -> 3
- net Col 11: track 251.6 -> 193.3 mm, vias 1 -> 3
- net Col 10: track 232.2 -> 175.1 mm, vias 1 -> 3
- net Col 6: track 151.2 -> 97.1 mm, vias 1 -> 2
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