File: LE75LRGB/LE75LRGB.kicad_pcb (KiCad board)
At the start: 2 copper layers, 285 x 94.6 mm, 256 parts, among them P1 USB_C_Plug_USB2.0, SW1 SW_Push, U1 MCP1703Ax-330xxDB, U2 STM32F072CBTx

Commit message: updated RGB variants
Routing:
- net GND: track 21.8 -> 33.6 mm, vias 216 -> 222
- net Net-(D120-DOUT): track 24.7 -> 28.2 mm
- net Row 0: track 327.9 -> 331.2 mm
- net Net-(D121-DOUT): track 22.2 -> 25.0 mm
- net RGB_addr: track 106.4 -> 109.0 mm
- net Net-(U2-BOOT0): track 47.6 -> 50.1 mm
- net Net-(D106-DIN): track 22.7 -> 25.2 mm
- net Net-(D76-DOUT): track 14.6 -> 16.4 mm
- net VCC: track 116.5 -> 117.8 mm
